File: PCBs/keyboard/dt-keyboard.kicad_pcb (KiCad board)
At the start: 2 copper layers, 87 parts

Commit message: Fixed Keyboard
Parts:
- moved J1 69.5 mm to (113.7, 57.4), turned to 0 degrees
Connections:
- J1 pad 10: Column 10 -> Column 6
- J1 pad 11: Row 0 -> Column 7
- J1 pad 12: Row 1 -> Column 8
- J1 pad 13: Row 2 -> Column 9
- J1 pad 14: Row 3 -> Column 10
- J1 pad 15: GND -> unconnected-(J1-MP-Pad15)
- J1 pad 16: GND -> unconnected-(J1-MP-Pad16)
- J1 pad 4: Column 4 -> Row 0
- J1 pad 5: Column 5 -> Row 1
- J1 pad 6: Column 6 -> Row 2
- J1 pad 7: Column 7 -> Row 3
- J1 pad 8: Column 8 -> Column 4
- J1 pad 9: Column 9 -> Column 5
Routing:
- net Column 10: track 271.5 -> 180.1 mm, vias 2 -> 0
- net Column 9: track 251.6 -> 161.7 mm, vias 2 -> 0
- net Column 8: track 229.2 -> 141.3 mm
- net Column 7: track 190.5 -> 104.8 mm
- net Column 6: track 195.6 -> 112.2 mm
- net Column 5: track 295.2 -> 214.4 mm
- net Column 4: track 159.9 -> 81.5 mm, vias 2 -> 0
- net Column 3: track 128.4 -> 81.3 mm, vias 2 -> 0
- net Column 0: track 90.6 -> 133.5 mm, vias 1 -> 0
- net Column 1: track 87.5 -> 118.9 mm
- net Row 1: track 282.5 -> 262.1 mm, vias 11 -> 12
- net Row 0: track 253.6 -> 235.1 mm
- net Row 3: track 376.4 -> 359.0 mm, vias 9 -> 10
- net Row 2: track 313.8 -> 296.8 mm, vias 11 -> 12
- net Column 2: track 111.4 -> 102.3 mm, vias 2 -> 0

Commit message: Layouting + Deep Sleep Tests
Parts:
- moved J1 31.4 mm to (82.5, 55.2)
Connections:
- J1 pad 3: Column 3 -> Row 0
- J1 pad 4: Row 0 -> Row 1
- J1 pad 5: Row 1 -> Row 2
- J1 pad 6: Row 2 -> Row 3
- J1 pad 7: Row 3 -> Column 3
Routing:
- net Column 4: track 81.5 -> 115.3 mm, vias 0 -> 2
- net Column 7: track 104.8 -> 137.2 mm
- net Column 6: track 112.2 -> 144.4 mm
- net Column 9: track 161.7 -> 193.7 mm
- net Column 8: track 141.3 -> 173.3 mm, vias 2 -> 0
- net Column 10: track 180.1 -> 211.7 mm
- net Column 5: track 214.4 -> 246.0 mm
- net Column 0: track 133.5 -> 102.0 mm
- net Column 1: track 118.9 -> 90.2 mm
- net Column 2: track 102.3 -> 77.1 mm
- net Row 3: track 359.0 -> 367.2 mm, vias 10 -> 9
- net Row 2: track 296.8 -> 304.3 mm, vias 12 -> 11
- net Column 3: track 81.3 -> 85.6 mm, vias 0 -> 2
- net Row 1: track 262.1 -> 264.0 mm, vias 12 -> 13

Commit message: Verification
Parts:
- added H1: MountingHole_Pad, MountingHole:MountingHole_3.2mm_M3_Pad_TopBottom, F.Cu at (41.1, 56.2)
- added H2: MountingHole_Pad, MountingHole:MountingHole_3.2mm_M3_Pad_TopBottom, F.Cu at (257.8, 56.2)
Other:
- board outline added: 231 x 88.1 mm
